Commit message: Update Crazyflie 2 model

File: rotors_description/urdf/crazyflie2.xacro (robot description, xacro)
@@ -22,5 +22,5 @@
   <xacro:property name="rotor_velocity_slowdown_sim" value="10" />
   <xacro:property name="use_mesh_file" value="true" />
-  <xacro:property name="mesh_file" value="package://rotors_description/meshes/hummingbird.dae" />
+  <xacro:property name="mesh_file" value="package://rotors_description/meshes/crazyflie2.dae" />
   <xacro:property name="mass" value="0.025" /> <!-- [kg] -->
   <xacro:property name="body_width" value="0.03" /> <!-- [m] -->
@@ -28,5 +28,5 @@
   <xacro:property name="mass_rotor" value="0.0005" /> <!-- [kg] -->
   <xacro:property name="arm_length" value="0.046" /> <!-- [m] -->
-  <xacro:property name="rotor_offset_top" value="0.029" /> <!-- [m] -->
+  <xacro:property name="rotor_offset_top" value="0.015" /> <!-- [m] -->
   <xacro:property name="radius_rotor" value="0.0225" /> <!-- [m] -->
   <xacro:property name="motor_constant" value="1.28192e-08" /> <!-- [kg m/s^2] -->

Commit message: Update Crazyflie 2 parameters and model

File: rotors_description/urdf/crazyflie2.xacro (robot description, xacro)
@@ -23,25 +23,26 @@
   <xacro:property name="use_mesh_file" value="true" />
   <xacro:property name="mesh_file" value="package://rotors_description/meshes/crazyflie2.dae" />
-  <xacro:property name="mass" value="0.025" /> <!-- [kg] -->
-  <xacro:property name="body_width" value="0.03" /> <!-- [m] -->
-  <xacro:property name="body_height" value="0.029" /> <!-- [m] -->
+  <xacro:property name="mass" value="0.024" /> <!-- [kg] -->
+  <xacro:property name="body_width" value="0.045" /> <!-- [m] -->
+  <xacro:property name="body_height" value="0.03" /> <!-- [m] -->
   <xacro:property name="mass_rotor" value="0.0005" /> <!-- [kg] -->
   <xacro:property name="arm_length" value="0.046" /> <!-- [m] -->
-  <xacro:property name="rotor_offset_top" value="0.015" /> <!-- [m] -->
+  <xacro:property name="rotor_offset_top" value="0.024" /> <!-- [m] -->
   <xacro:property name="radius_rotor" value="0.0225" /> <!-- [m] -->
+  <!-- Forster's -->
   <xacro:property name="motor_constant" value="1.28192e-08" /> <!-- [kg m/s^2] -->
   <xacro:property name="moment_constant" value="5.964552e-03" /> <!-- [m] -->
   <xacro:property name="time_constant_up" value="0.0125" /> <!-- [s] -->
   <xacro:property name="time_constant_down" value="0.025" /> <!-- [s] -->
-  <xacro:property name="max_rot_velocity" value="3052" /> <!-- [rad/s] -->
+  <xacro:property name="max_rot_velocity" value="2618" /> <!-- [rad/s] -->
   <xacro:property name="rotor_drag_coefficient" value="8.06428e-05" />
   <xacro:property name="rolling_moment_coefficient" value="0.000001" />
   <!-- Property Blocks -->
   <xacro:property name="body_inertia">
-    <inertia ixx="0.01152" ixy="0.0" ixz="0.0" iyy="0.01152" iyz="0.0" izz="0.0218" /> <!-- [kg m^2] [kg m^2] [kg m^2] [kg m^2] [kg m^2] [kg m^2] -->
+    <inertia ixx="1.657171e-05" ixy="0.0" ixz="0.0" iyy="1.657171e-05" iyz="0.0" izz="2.9261652e-05" />
   </xacro:property>
   <!-- inertia of a single rotor, assuming it is a cuboid. Height=0.4mm, width=0.8mm -->
   <xacro:property name="rotor_inertia">
-    <xacro:box_inertia x="${radius_rotor}" y="0.0008" z="0.0004" mass="${mass_rotor*rotor_velocity_slowdown_sim}" />
+    <xacro:box_inertia x="${radius_rotor}" y="0.007" z="0.003" mass="${mass_rotor*rotor_velocity_slowdown_sim}" />
   </xacro:property>
   <!-- Included URDF Files -->

File: rotors_description/urdf/crazyflie2_base.xacro (robot description, xacro)
@@ -32,5 +32,5 @@
       parent_link="${namespace}/base_link"
       imu_topic="imu"
-      mass_imu_sensor="0.002"
+      mass_imu_sensor="0.001"
       gyroscope_noise_density="0.0003394"
       gyroscopoe_random_walk="0.000038785"
